Commit message: removed dependency from the IMAV package

File: urdf/quadrotor.urdf.xacro (robot description, xacro)
@@ -6,29 +6,29 @@
     <!-- Included URDF Files -->
     <!-- Base airframe -->
-    <xacro:include filename="$(find imav_2017)/urdf/quadrotor_base.urdf.xacro" />
+    <xacro:include filename="$(find viscap_gazebo)/urdf/quadrotor_base.urdf.xacro" />
     <quadrotor_base_macro/>
     <!-- IMU, Baro, Magnetic, GPS, Groundtruth sensors -->
-    <xacro:include filename="$(find imav_2017)/urdf/sensors/quadrotor_sensors.urdf.xacro" />
+    <xacro:include filename="$(find viscap_gazebo)/urdf/sensors/quadrotor_sensors.urdf.xacro" />
     <quadrotor_sensors robot_name="${robot_name}"/>
     <!-- 4D velocity control -->
-    <xacro:include filename="$(find imav_2017)/urdf/quadrotor_simple_controller.urdf.xacro" />
+    <xacro:include filename="$(find viscap_gazebo)/urdf/quadrotor_simple_controller.urdf.xacro" />
     <quadrotor_controller robot_name="${robot_name}"/>
     <!-- Sonar height sensor -->
-    <xacro:include filename="$(find imav_2017)/urdf/sensors/sonar_sensor.urdf.xacro" />
+    <xacro:include filename="$(find viscap_gazebo)/urdf/sensors/sonar_sensor.urdf.xacro" />
     <xacro:sonar_sensor name="sonar" parent="base_link" sim_name="${robot_name}" ros_topic="sonar_height" update_rate="10" min_range="0.01" max_range="3.0" field_of_view="${40*M_PI/180}" ray_count="3">
       <origin xyz="-0.15 0.0 0.0" rpy="0 ${90*M_PI/180} 0"/>
     </xacro:sonar_sensor>
     <!-- Hokuyo UTM-30LX mounted upside down below the quadrotor body -->
-    <xacro:include filename="$(find imav_2017)/urdf/sensors/hokuyo_utm30lx.urdf.xacro" />
+    <xacro:include filename="$(find viscap_gazebo)/urdf/sensors/hokuyo_utm30lx.urdf.xacro" />
     <xacro:hokuyo_utm30lx name="laser0" robot_name="${robot_name}" parent="base_link" ros_topic="scan" update_rate="40" ray_count="1081" min_angle="135" max_angle="-135">
       <origin xyz="0.0 0.0 0.08" rpy="${M_PI} 0 0"/>
     </xacro:hokuyo_utm30lx>
     <!-- Forward facing camera -->
-    <xacro:include filename="$(find imav_2017)/urdf/sensors/generic_camera.urdf.xacro" />
+    <xacro:include filename="$(find viscap_gazebo)/urdf/sensors/generic_camera.urdf.xacro" />
     <xacro:generic_camera name="front" sim_name="${robot_name}" parent="base_link" update_rate="60" res_x="640" res_y="360" image_format="R8G8B8" hfov="${81*M_PI/180}">
       <origin xyz="0.21 0.0 0.01" rpy="0 0 0"/>
     </xacro:generic_camera>
     <!-- Downward facing camera -->
-    <xacro:include filename="$(find imav_2017)/urdf/sensors/generic_camera.urdf.xacro" />
+    <xacro:include filename="$(find viscap_gazebo)/urdf/sensors/generic_camera.urdf.xacro" />
     <xacro:generic_camera name="bottom" sim_name="${robot_name}" parent="base_link" update_rate="60" res_x="640" res_y="360" image_format="R8G8B8" hfov="${81*M_PI/180}">
       <origin xyz="0.15 0.0 0.0" rpy="0 ${M_PI/2} 0"/>

File: urdf/quadrotor_base.urdf.xacro (robot description, xacro)
@@ -13,5 +13,5 @@
         <origin xyz="0 0 0" rpy="0 0 0" />
         <geometry>
-          <mesh filename="package://imav_2017/meshes/quadrotor/quadrotor_4.dae"/>
+          <mesh filename="package://viscap_gazebo/meshes/quadrotor/quadrotor_4.dae"/>
         </geometry>
       </visual>
@@ -19,5 +19,5 @@
         <origin xyz="0 0 0" rpy="0 0 0" />
         <geometry>
-          <mesh filename="package://imav_2017/meshes/quadrotor/quadrotor_4.stl"/>
+          <mesh filename="package://viscap_gazebo/meshes/quadrotor/quadrotor_4.stl"/>
         </geometry>
       </collision>

File: urdf/sensors/hokuyo_utm30lx.urdf.xacro (robot description, xacro)
@@ -16,5 +16,5 @@
 	  <origin xyz="0 0 0" rpy="0 0 0" />
           <geometry>
-          <mesh filename="package://imav_2017/meshes/hokuyo_utm30lx/hokuyo_utm_30lx$(optenv TEST_SELF_FILTER).dae"/>
+          <mesh filename="package://viscap_gazebo/meshes/hokuyo_utm30lx/hokuyo_utm_30lx$(optenv TEST_SELF_FILTER).dae"/>
         </geometry>
 	</visual>

File: urdf/sensors/sonar_sensor.urdf.xacro (robot description, xacro)
@@ -17,5 +17,5 @@
         <geometry>
           <!--<box size="0.01 0.01 0.01" /> -->
-          <mesh filename="package://imav_2017/meshes/sonar_sensor/max_sonar_ez4.dae"/>
+          <mesh filename="package://viscap_gazebo/meshes/sonar_sensor/max_sonar_ez4.dae"/>
         </geometry>
       </visual>

File: worlds/xacro/imav_indoor.world.xacro (robot description, xacro)
@@ -6,5 +6,4 @@
     <xacro:property name="length2" value="10" />
     <xacro:property name="length3" value="13" />
-    <!--xacro:include filename="$(find imav_2017)/worlds/xacro/macros.urdf.xacro" /-->
     <xacro:include filename="macros.urdf.xacro" />
     <xacro:light_source/>

File: worlds/xacro/macros.urdf.xacro (robot description, xacro)
@@ -149,5 +149,5 @@
           <material>
             <script>
-              <uri>file://$(find imav_2017)/worlds/xacro/custom.material</uri>
+              <uri>file://$(find viscap_gazebo)/worlds/xacro/custom.material</uri>
               <name>MathWorks_branding</name>
             </script>
@@ -194,5 +194,5 @@
             <geometry>
               <mesh>
-                <uri>file://$(find imav_2017)/worlds/xacro/wall.dae</uri>
+                <uri>file://$(find viscap_gazebo)/worlds/xacro/wall.dae</uri>
                 <scale>0.1 0.1 0.1</scale>
               </mesh>
@@ -208,5 +208,5 @@
             <geometry>
               <mesh>
-                <uri>file://$(find imav_2017)/worlds/xacro/wall.dae</uri>
+                <uri>file://$(find viscap_gazebo)/worlds/xacro/wall.dae</uri>
                 <scale>0.1 0.1 0.1</scale>
               </mesh>
@@ -339,5 +339,5 @@
             <geometry>
               <mesh>
-                <uri>file://$(find imav_2017)/worlds/xacro/tree1.dae</uri>
+                <uri>file://$(find viscap_gazebo)/worlds/xacro/tree1.dae</uri>
                 <scale>0.01 0.01 0.01</scale>
               </mesh>
@@ -348,5 +348,5 @@
             <geometry>
               <mesh>
-                <uri>file://$(find imav_2017)/worlds/xacro/tree1.dae</uri>
+                <uri>file://$(find viscap_gazebo)/worlds/xacro/tree1.dae</uri>
                 <scale>0.01 0.01 0.01</scale>
               </mesh>
@@ -374,5 +374,5 @@
             <geometry>
               <mesh>
-                <uri>file://$(find imav_2017)/worlds/xacro/tree1.dae</uri>
+                <uri>file://$(find viscap_gazebo)/worlds/xacro/tree1.dae</uri>
                 <scale>0.01 0.004 0.01</scale>
               </mesh>
@@ -383,5 +383,5 @@
             <geometry>
               <mesh>
-                <uri>file://$(find imav_2017)/worlds/xacro/tree1.dae</uri>
+                <uri>file://$(find viscap_gazebo)/worlds/xacro/tree1.dae</uri>
                 <scale>0.01 0.004 0.01</scale>
               </mesh>
@@ -426,5 +426,5 @@
         <material>
           <script>
-            <uri>file://$(find imav_2017)/worlds/xacro/custom.material</uri>
+            <uri>file://$(find viscap_gazebo)/worlds/xacro/custom.material</uri>
             <name>Helipad</name>
           </script>
@@ -500,5 +500,5 @@
           <material>
             <script>
-              <uri>file://$(find imav_2017)/worlds/xacro/custom.material</uri>
+              <uri>file://$(find viscap_gazebo)/worlds/xacro/custom.material</uri>
               <name>QR1</name>
             </script>
@@ -536,5 +536,5 @@
           <material>
             <script>
-              <uri>file://$(find imav_2017)/worlds/xacro/custom.material</uri>
+              <uri>file://$(find viscap_gazebo)/worlds/xacro/custom.material</uri>
               <name>X1</name>
             </script>
